File: power_p16.kicad_pcb (KiCad board)
At the start: 4 copper layers, 44.8 x 41.5 mm, 23 parts, among them J1 LSHM-140-04.0-L-DV-A-N-K-TR, U1 LT8350S

Commit message: Update
Connections:
- J1 pad 52: 16V -> GND
- J1 pad 54: 16V -> GND
- J1 pad 56: 16V -> GND
- J1 pad 58: 16V -> GND
- J1 pad 60: 16V -> GND
- J1 pad 62: GND -> 16V
- J1 pad 64: GND -> 16V
- J1 pad 66: GND -> 16V
- J1 pad 68: GND -> 16V
- J1 pad 70: GND -> 16V
Routing:
- net 16V: track 62.8 -> 65.7 mm
- net GND: vias 156 -> 155
Changed lines of the file:
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@@
 			(size 0.3 1.5)
 			(layers "B.Cu" "B.Mask" "B.Paste")
-			(net 5 "16V")
+			(net 1 "GND")
 			(pinfunction "Pin_52")
 			(pintype "passive")
@@
 			(size 0.3 1.5)
 			(layers "B.Cu" "B.Mask" "B.Paste")
-			(net 5 "16V")
+			(net 1 "GND")
 			(pinfunction "Pin_54")
 			(pintype "passive")
@@
 			(size 0.3 1.5)
 			(layers "B.Cu" "B.Mask" "B.Paste")
-			(net 5 "16V")
+			(net 1 "GND")
 			(pinfunction "Pin_56")
 			(pintype "passive")
@@
 			(size 0.3 1.5)
 			(layers "B.Cu" "B.Mask" "B.Paste")
-			(net 5 "16V")
+			(net 1 "GND")
 			(pinfunction "Pin_58")
 			(pintype "passive")
@@
 			(size 0.3 1.5)
 			(layers "B.Cu" "B.Mask" "B.Paste")
-			(net 5 "16V")
+			(net 1 "GND")
 			(pinfunction "Pin_60")
 			(pintype "passive")
@@
 			(size 0.3 1.5)
 			(layers "B.Cu" "B.Mask" "B.Paste")
-			(net 1 "GND")
+			(net 5 "16V")
 			(pinfunction "Pin_62")
 			(pintype "passive")
@@
 			(size 0.3 1.5)
 			(layers "B.Cu" "B.Mask" "B.Paste")
-			(net 1 "GND")
+			(net 5 "16V")
 			(pinfunction "Pin_64")
 			(pintype "passive")
@@
 			(size 0.3 1.5)
 			(layers "B.Cu" "B.Mask" "B.Paste")
-			(net 1 "GND")
+			(net 5 "16V")
 			(pinfunction "Pin_66")
 			(pintype "passive")
@@
 			(size 0.3 1.5)
 			(layers "B.Cu" "B.Mask" "B.Paste")
-			(net 1 "GND")
+			(net 5 "16V")
 			(pinfunction "Pin_68")
 			(pintype "passive")
@@
 			(size 0.3 1.5)
 			(layers "B.Cu" "B.Mask" "B.Paste")
-			(net 1 "GND")
+			(net 5 "16V")
 			(pinfunction "Pin_70")
 			(pintype "passive")
@@
 	)
 	(via
-		(at 52.65 28.65)
+		(at 55.3 27.6)
 		(size 0.6)
 		(drill 0.3)
@@
 	)
 	(via
-		(at 56.1 28.85)
+		(at 56.6 29)
 		(size 0.6)
 		(drill 0.3)
@@
 	)
 	(via
-		(at 54.9 26.6)
-		(size 0.6)
-		(drill 0.3)
-		(layers "F.Cu" "B.Cu")
-		(free yes)
-		(net 1)
-	)
-	(via
 		(at 37.6 63.1)
 		(size 0.6)
@@
 	)
 	(via
-		(at 51.25 26.9)
+		(at 53.5 26.4)
 		(size 0.6)
 		(drill 0.3)
@@
 	)
 	(segment
-		(start 50.15 30.6)
-		(end 50.15 29.25)
-		(width 2.3)
-		(layer "B.Cu")
-		(net 5)
-	)
-	(segment
-		(start 49 28.1)
-		(end 34.55 28.1)
+		(start 34.55 28.1)
+		(end 52.252 28.1)
 		(width 2.3)
 		(layer "B.Cu")
@@
 	)
 	(segment
-		(start 50.15 29.25)
-		(end 49 28.1)
-		(width 2.3)
-		(layer "B.Cu")
-		(net 5)
-	)
-	(segment
 		(start 47.100498 42.549)
 		(end 44.651 42.549)
@@
 	)
 	(segment
+		(start 52.65 28.498)
+		(end 52.65 30.6)
+		(width 2.3)
+		(layer "B.Cu")
+		(net 5)
+	)
+	(segment
 		(start 38.8 45.2)
 		(end 35.8 48.2)
@@
 		(layer "B.Cu")
 		(net 5)
+	)
+	(segment
+		(start 52.252 28.1)
+		(end 52.65 28.498)
+		(width 2.3)
+		(layer "B.Cu")
+		(net 5)
